Commit message: modified according to requirements

File: fairino5_v6_moveit2_config/config/fairino5_v6_robot.ros2_control.xacro (robot description, xacro)
@@ -1,10 +1,16 @@
 <?xml version="1.0"?>
 <robot xmlns:xacro="http://www.ros.org/wiki/xacro">
-    <xacro:macro name="fairino5_v6_robot_ros2_control" params="name initial_positions_file">
+    <xacro:macro name="fairino5_v6_robot_ros2_control" params="name initial_positions_file use_hardware">
         <xacro:property name="initial_positions" value="${load_yaml(initial_positions_file)['initial_positions']}"/>
+        <!-- Normalize boolean-ish arg to a strict boolean -->
+        <xacro:property name="use_hw" value="${use_hardware in ['true','True','1',1,True]}"/>
         <ros2_control name="${name}" type="system">
             <hardware>
-                <!-- By default, set up controllers for simulation. This won't work on real hardware -->
-                <plugin>mock_components/GenericSystem</plugin>
+                <xacro:if value="${use_hw}">
+                    <plugin>fairino_hardware/FairinoHardwareInterface</plugin>
+                </xacro:if>
+                <xacro:unless value="${use_hw}">
+                    <plugin>mock_components/GenericSystem</plugin>
+                </xacro:unless>
             </hardware>
             <joint name="j1">

File: fairino5_v6_moveit2_config/config/fairino5_v6_robot.urdf.xacro (robot description, xacro)
@@ -2,8 +2,18 @@
 <robot xmlns:xacro="http://www.ros.org/wiki/xacro" name="fairino5_v6_robot">
     <xacro:arg name="initial_positions_file" default="initial_positions.yaml" />
+    <xacro:arg name="use_hardware" default="false" />
+    <xacro:arg name="use_realsense" default="false" />
     <!-- Import fairino5_v6_robot urdf file -->
     <xacro:include filename="$(find fairino_description)/urdf/fairino5_v6.urdf" />
+    <!-- Include RealSense D435i camera description (camera-only xacro) - optional -->
+    <xacro:if value="$(arg use_realsense)">
+        <xacro:include filename="$(find realsense2_description)/urdf/_d435i.urdf.xacro" />
+        <!-- Instantiate D435i camera and attach to weld mount connector link -->
+        <xacro:sensor_d435i parent="weld_mount_connector_link">
+            <origin xyz="0 0.0605 0.01415" rpy="0 -1.57079632679 -1.57079632679"/>
+        </xacro:sensor_d435i>
+    </xacro:if>
     <!-- Import control_xacro -->
     <xacro:include filename="fairino5_v6_robot.ros2_control.xacro" />
-    <xacro:fairino5_v6_robot_ros2_control name="FakeSystem" initial_positions_file="$(arg initial_positions_file)"/>
+    <xacro:fairino5_v6_robot_ros2_control name="FakeSystem" initial_positions_file="$(arg initial_positions_file)" use_hardware="$(arg use_hardware)"/>
 </robot>
