Commit message: modified robot_description

File: fairino_description/urdf/fairino5_v6.urdf (robot description, URDF)
Before this commit: robot fairino5_v6_robot, 7 links, 6 joints
Links:
- added link weld_mount_connector_link; collision mesh filename=package://fairino_description/meshes/fairino5_v6/weld_end_e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; visual mesh filename=package://fairino_description/meshes/fairino5_v6/weld_end_e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
- added link weld_tip
Joints:
- added joint weld_mount_connector_to_weld_tip: type fixed, parent weld_mount_connector_link, child weld_tip, origin xyz=0 0.04868120 0.25567253 rpy=0 0 0
- added joint wrist3_to_weld_mount_connector: type fixed, parent wrist3_link, child weld_mount_connector_link, origin xyz=0 0 0.0911 rpy=0 0 3.14159
